Commit message: work with keyboard

File: src/diffbot_description/urdf/diffbot.urdf (robot description, URDF)
Before this commit: robot diffbot, 3 links, 2 joints
Links:
- link base_link: mass 5.0 -> 6.0
- link left_wheel: mass None -> 0.3; geometry collision cylinder length=0.03 radius=0.05; visual cylinder length=0.03 radius=0.05
- link right_wheel: mass None -> 0.3; geometry collision cylinder length=0.03 radius=0.05; visual cylinder length=0.03 radius=0.05
Joints:
- joint left_wheel_joint: origin xyz=0 0.15 0 -> xyz=0 0.15 -0.05
- joint right_wheel_joint: origin xyz=0 -0.15 0 -> xyz=0 -0.15 -0.05

Commit message: fixe Dockerfile

File: src/diffbot_description/urdf/diffbot.urdf (robot description, URDF)
Before this commit: robot diffbot, 3 links, 2 joints
Links:
- link left_wheel: geometry collision cylinder length=0.01 radius=0.0285; visual cylinder length=0.01 radius=0.0285
- link right_wheel: geometry collision cylinder length=0.01 radius=0.0285; visual cylinder length=0.01 radius=0.0285
Joints:
- joint left_wheel_joint: origin xyz=0 0.15 -0.05 -> xyz=0 0.15 -0.03
- joint right_wheel_joint: origin xyz=0 -0.15 -0.05 -> xyz=0 -0.15 -0.03
