Commit message: commit pour Thoru

File: src/eirbot2026/urdf/eirbot2026.urdf.xacro (robot description, xacro)
@@ -23,16 +23,21 @@
     <link name="base">
         <collision>
-            <origin xyz="0 0 0.05" rpy="0 0 0" />
+            <origin xyz="0 0 0.3" rpy="0 0 0" />
             <geometry>
-                <box size="3.0 3.0 0.1" />
+                <box size="1 0.5 0.3" />
             </geometry>
         </collision>
         <visual>
-            <origin xyz="0 0 0.05" rpy="0 0 0" />
+            <origin xyz="0 0 0.3" rpy="0 0 0" />
             <geometry>
-                <box size="3.0 3.0 0.1" />
+                <box size="1 0.5 0.3" />
             </geometry>
             <material name="green" />
         </visual>
+        <inertial>
+            <mass value = "1.0" />
+            <inertia ixx = "0.01" ixy = "0.0" ixz = "0.0"
+                     iyy = "0.01" iyz = "0.0" izz = "0.01" />
+        </inertial>
     </link>
     <!-- Define link named "rotor1" -->
@@ -41,5 +46,5 @@
             <origin xyz="0 0 0" rpy="0 0 0" />
             <geometry>
-                <cylinder radius="0.3" length="0.5" />
+                <cylinder radius="0.3" length="0.1" />
             </geometry>
         </collision>
@@ -47,8 +52,13 @@
             <origin xyz="0 0 0" rpy="0 0 0" />
             <geometry>
-                <cylinder radius="0.3" length="0.5" />
+                <cylinder radius="0.3" length="0.1" />
             </geometry>
             <material name="red" />
         </visual>
+        <inertial>
+            <mass value = "1.0" />
+            <inertia ixx = "0.01" ixy = "0.0" ixz = "0.0"
+                     iyy = "0.01" iyz = "0.0" izz = "0.01" />
+        </inertial>
     </link>
     <!-- Define link named "rotor2" -->
@@ -57,5 +67,5 @@
             <origin xyz="0 0 0" rpy="0 0 0" />
             <geometry>
-                <cylinder radius="0.3" length="0.5" />
+                <cylinder radius="0.3" length="0.1" />
             </geometry>
         </collision>
@@ -63,8 +73,13 @@
             <origin xyz="0 0 0" rpy="0 0 0" />
             <geometry>
-                <cylinder radius="0.3" length="0.5" />
+                <cylinder radius="0.3" length="0.1" />
             </geometry>
             <material name="red" />
         </visual>
+        <inertial>
+            <mass value = "1.0" />
+            <inertia ixx = "0.01" ixy = "0.0" ixz = "0.0"
+                     iyy = "0.01" iyz = "0.0" izz = "0.01" />
+        </inertial>
     </link>
     <!-- Define joint named "joint1" with type "fixed" -->
@@ -79,5 +94,5 @@
         <parent link="base" />
         <child link="rotor1" />
-        <origin xyz="0.325 0 0.25" rpy="-0.5236 0 0" />
+        <origin xyz="-0.25 0.5 0.25" rpy="-1.5236 0 0" />
         <axis xyz="0 0 1" />
     </joint>
@@ -86,5 +101,5 @@
         <parent link="base" />
         <child link="rotor2" />
-        <origin xyz="-0.325 0 0.25" rpy="-0.5236 0 0" />
+        <origin xyz="-0.25 -0.5 0.25" rpy="-1.5236 0 0" />
         <axis xyz="0 0 1" />
     </joint>
