Commit message: Starting to abandon gazebo

File: src/diffdrive_arduino-humble/description/ros2_control/diffbot.ros2_control.xacro (robot description, xacro)
@@ -34,4 +34,10 @@
       </joint>
     </ros2_control>
+    <hardware>
+      <xacro:if value="$(arg use_mock)">
+        <plugin>mock_components/GenericSystem</plugin>
+        <param name="calculate_dynamics">true</param>
+      </hardware>
+    </hardware>
   </xacro:macro>
 </robot>

File: src/diffdrive_arduino-humble/description/urdf/diffbot_description.urdf.xacro (robot description, xacro)
@@ -4,5 +4,5 @@
   <!-- Constants for robot dimensions -->
   <xacro:property name="PI" value="3.1415926535897931"/>
-  <xacro:property name="base_mass" value="0.3" /> <!-- arbitrary value for base mass -->
+  <xacro:property name="base_mass" value="5" /> <!-- arbitrary value for base mass -->
   <xacro:property name="base_width" value="0.1" />
   <xacro:property name="base_length" value="0.1" />
@@ -11,5 +11,5 @@
   <xacro:property name="wheel_len" value="0.020" />
   <xacro:property name="wheel_radius" value="0.015" />
-  <xacro:property name="caster_wheel_mass" value="0.1" /> <!-- arbitrary value for caster wheel mass -->
+  <xacro:property name="caster_wheel_mass" value="0.2" /> <!-- arbitrary value for caster wheel mass -->
   <xacro:property name="caster_wheel_radius" value="0.015" />
   <xacro:property name="z_offset" value="-${base_height/2}" /> <!-- Space btw top of beam and the each joint -->

Commit message: don' know the name

File: src/diffdrive_arduino-humble/description/ros2_control/diffbot.ros2_control.xacro (robot description, xacro)
@@ -1,25 +1,23 @@
 <?xml version="1.0"?>
 <robot xmlns:xacro="http://www.ros.org/wiki/xacro">
-  <xacro:arg name="use_gazebo" default="false" />
-  <xacro:macro name="diffbot_ros2_control" params="name prefix">
+  <xacro:macro name="diffbot_ros2_control" params="name prefix use_mock:=true use_gazebo:=false">
     <ros2_control name="${name}" type="system">
       <hardware>
-        <xacro:if value="$(arg use_gazebo)">
-          <plugin>gazebo_ros2_control/GazeboSystem</plugin>
+        <xacro:if value="${use_mock}">
+          <plugin>mock_components/GenericSystem</plugin>
+          <param name="calculate_dynamics">true</param>
         </xacro:if>
-        <xacro:unless value="$(arg use_gazebo)">
-          <plugin>diffdrive_arduino/DiffDriveArduinoHardware</plugin>
-          <param name="left_wheel_name">left_wheel_joint</param>
-          <param name="right_wheel_name">right_wheel_joint</param>
-          <param name="loop_rate">30</param>
-          <param name="device">/dev/serial/by-path/platform-fd500000.pcie-pci-0000:01:00.0-usb-0:1.3:1.0-port0</param>
-          <param name="baud_rate">57600</param>
-          <param name="timeout_ms">1000</param>
-          <param name="enc_counts_per_rev">3436</param>
+        <xacro:unless value="${use_mock}">
+          <xacro:unless value="${use_gazebo}">
+            <plugin>diffdrive_arduino/DiffDriveArduinoHardware</plugin>
+            <param name="left_wheel_name">${prefix}left_wheel_joint</param>
+            <param name="right_wheel_name">${prefix}right_wheel_joint</param>
+            <param name="loop_rate">30</param>
+            <param name="device">/dev/serial/by-path/platform-fd500000.pcie-pci-0000:01:00.0-usb-0:1.3:1.0-port0</param>
+            <param name="baud_rate">57600</param>
+            <param name="timeout_ms">1000</param>
+            <param name="enc_counts_per_rev">3436</param>
+          </xacro:unless>
         </xacro:unless>
-        <param name="pid_p">20</param>
-        <param name="pid_d">12</param>
-        <param name="pid_i">0</param>
-        <param name="pid_o">50</param>
       </hardware>
       <joint name="${prefix}left_wheel_joint">
@@ -34,10 +32,4 @@
       </joint>
     </ros2_control>
-    <hardware>
-      <xacro:if value="$(arg use_mock)">
-        <plugin>mock_components/GenericSystem</plugin>
-        <param name="calculate_dynamics">true</param>
-      </hardware>
-    </hardware>
   </xacro:macro>
 </robot>

File: src/diffdrive_arduino-humble/description/urdf/diffbot.urdf.xacro (robot description, xacro)
@@ -2,4 +2,5 @@
 <!-- Basic differential drive mobile base -->
 <robot xmlns:xacro="http://www.ros.org/wiki/xacro" name="diffdrive_robot">
+  <xacro:arg name="use_mock" default="true" />
   <xacro:arg name="prefix" default="" />
   <xacro:include filename="$(find diffdrive_arduino)/urdf/diffbot_description.urdf.xacro" />
@@ -10,9 +11,6 @@
   <xacro:diffbot prefix="$(arg prefix)" />
   <xacro:diffbot_ros2_control
-    name="DiffBot" prefix="$(arg prefix)" />
-  <gazebo>
-      <plugin name="gazebo_ros2_control" filename="libgazebo_ros2_control.so">
-          <parameters>$(find diffdrive_arduino)/config/diffbot_controllers.yaml</parameters>
-      </plugin>
-  </gazebo>
+    name="DiffBot"
+    prefix=""
+    use_mock="$(arg use_mock)" />
 </robot>
