Commit message: hhh

File: src/diffdrive_arduino-humble/description/urdf/diffbot_description.urdf.xacro (robot description, xacro)
@@ -5,12 +5,12 @@
   <xacro:property name="PI" value="3.1415926535897931"/>
   <xacro:property name="base_mass" value="5" /> <!-- arbitrary value for base mass -->
-  <xacro:property name="base_width" value="0.1" />
-  <xacro:property name="base_length" value="0.1" />
-  <xacro:property name="base_height" value="0.05" />
+  <xacro:property name="base_width" value="0.36" />
+  <xacro:property name="base_length" value="0.33" />
+  <xacro:property name="base_height" value="0.35" />
   <xacro:property name="wheel_mass" value="0.3" /> <!-- arbitrary value for wheel mass -->
-  <xacro:property name="wheel_len" value="0.020" />
-  <xacro:property name="wheel_radius" value="0.015" />
+  <xacro:property name="wheel_len" value="0.010" />
+  <xacro:property name="wheel_radius" value="0.020" />
   <xacro:property name="caster_wheel_mass" value="0.2" /> <!-- arbitrary value for caster wheel mass -->
-  <xacro:property name="caster_wheel_radius" value="0.015" />
+  <xacro:property name="caster_wheel_radius" value="0.020" />
   <xacro:property name="z_offset" value="-${base_height/2}" /> <!-- Space btw top of beam and the each joint -->
   <!-- Base Link -->

Commit message: more obstacles

File: src/diffdrive_arduino-humble/description/urdf/diffbot_description.urdf.xacro (robot description, xacro)
@@ -17,5 +17,5 @@
   <link name="${prefix}base_link">
     <collision>
-      <origin xyz="0 0 0" rpy="0 0 0"/>
+      <origin xyz="0 0 ${base_height/2}" rpy="0 0 0"/>
       <geometry>
         <box size="${base_width} ${base_length} ${base_height}"/>
@@ -23,5 +23,5 @@
     </collision>
     <visual>
-      <origin xyz="0 0 ${base_height/2}" rpy="0 0 0"/>
+      <origin xyz="0 0 0" rpy="0 0 0"/>
       <geometry>
         <box size="${base_width} ${base_length} ${base_height}"/>
@@ -158,4 +158,30 @@
         </inertial>
       </link>
+      <!-- ****************************** LIDAR *****************************    -->
+      <joint name="${prefix}lidar_joint" type="fixed">
+        <parent link="${prefix}base_link"/>
+        <child link="${prefix}lidar_link"/>
+        <origin xyz="0 0 ${base_height}" rpy="0 0 0"/>
+      </joint>
+      <link name="${prefix}lidar_link">
+        <inertial>
+          <mass value="0.1"/>
+          <origin xyz="0 0 0" rpy="0 0 0"/>
+          <inertia ixx="0.0001" ixy="0" ixz="0" iyy="0.0001" iyz="0" izz="0.0001"/>
+        </inertial>
+        <collision>
+          <origin xyz="0 0 0" rpy="0 0 0"/>
+          <geometry>
+            <cylinder radius="0.0508" length="0.18"/>
+          </geometry>
+        </collision>
+        <visual>
+          <origin xyz="0 0 0" rpy="0 0 0"/>
+          <geometry>
+            <cylinder radius="0.0508" length="0.18"/>
+          </geometry>
+          <material name="black"/>
+        </visual>
+      </link>
   </xacro:macro>
 </robot>
