Commit message: done eirbot_base

File: src/eirbot_base/description/ros2_control/robot.ros2_control.xacro (robot description, xacro)
@@ -1,5 +1,5 @@
 <?xml version="1.0"?>
 <robot xmlns:xacro="http://www.ros.org/wiki/xacro">
-  <xacro:macro name="diffbot_ros2_control" params="name prefix use_mock:=true use_gazebo:=false">
+  <xacro:macro name="eirbot_ros2_control" params="name prefix use_mock:=true use_gazebo:=false">
     <ros2_control name="${name}" type="system">
       <hardware>
@@ -10,5 +10,5 @@
         <xacro:unless value="${use_mock}">
           <xacro:unless value="${use_gazebo}">
-            <plugin>diffdrive_arduino/DiffBotMicroRos</plugin>
+            <plugin>eirbot_base/EirbotMicroRos</plugin>
             <param name="left_wheel_name">${prefix}left_wheel_joint</param>
             <param name="right_wheel_name">${prefix}right_wheel_joint</param>

File: src/eirbot_base/description/urdf/robot_description.urdf.xacro (robot description, xacro)
@@ -1,5 +1,5 @@
 <?xml version="1.0"?>
 <robot xmlns:xacro="http://www.ros.org/wiki/xacro">
-  <xacro:macro name="diffbot" params="prefix">
+  <xacro:macro name="eirbot_base" params="prefix">
   <!-- Constants for robot dimensions -->
   <xacro:property name="PI" value="3.1415926535897931"/>
